File: Jornada_keyboard_USB v.3/Jornada_keyboard_USB.kicad_sch (KiCad schematic)
At the start: 26 parts, among them J1 Conn_01x01_Socket, J2 USB_B_Micro, J3 Conn_01x24_MountingPin, J4 Conn_01x01_Socket, J5 Conn_01x01_Socket, J6 Conn_01x01_Socket, J7 Conn_01x01_Socket, J8 Conn_01x01_Socket, SW1 SW_Omron_B3FS, U1 ATmega32U4-A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

Commit message: Add files via upload
Parts:
- R5: value R -> 860
Changed lines of the file:
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@@
 			)
 		)
-		(property "Value" "R"
+		(property "Value" "860"
 			(at 68.58 124.4599 0)
 			(effects
